File: CPU.kicad_sch (KiCad schematic)
At the start: 4 parts, among them U28 NUCLEO-L152RE

Commit message: alueet laatikoitu, ensimmäiset input osat laitettu
Changed lines of the file:
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@@
 	(paper "A4")
 	(rectangle
-		(start 46.99 50.8)
-		(end 195.58 140.97)
+		(start 46.99 24.13)
+		(end 209.55 140.97)
 		(stroke
 			(width 0)
@@
 		)
 		(fill
-			(type none)
-		)
-	)
-	(rectangle
-		(start 149.86 24.13)
-		(end 212.09 49.53)
-		(stroke
-			(width 0)
-			(type default)
-			(color 252 0 255 1)
-		)
-		(fill
