File: Communication.kicad_sch (KiCad schematic)
At the start: 5 parts, among them J15 Screw_Terminal_01x03, U27 ADM2483xRW

Commit message: alueet laatikoitu, ensimmäiset input osat laitettu
Changed lines of the file:
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@@
 	(generator_version "9.0")
 	(paper "A4")
+	(rectangle
+		(start 95.25 63.5)
+		(end 151.13 133.35)
+		(stroke
+			(width 0)
+			(type default)
+			(color 255 0 249 1)
+		)
+		(fill
+			(type none)
+		)
+	)
+	(rectangle
+		(start 151.13 63.5)
+		(end 210.82 133.35)
+		(stroke
+			(width 0)
+			(type default)
+			(color 251 0 255 1)
+		)
+		(fill
+			(type none)
+		)
+	)
 	(text "RS-485 \n(Modbus-RTU)\n"
 		(exclude_from_sim no)
