File: DO.kicad_sch (KiCad schematic)
At the start: 50 parts, among them J3 Screw_Terminal_01x02, J4 Screw_Terminal_01x02, J5 Screw_Terminal_01x02, J6 Screw_Terminal_01x02, K1 SDT-S-103DMR,000, K2 SDT-S-103DMR,000, K3 SDT-S-103DMR,000, K4 SDT-S-103DMR,000, Q13 AO3400A, Q7 AO3400A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

Commit message: alueet laatikoitu, ensimmäiset input osat laitettu
Changed lines of the file:
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@@
 	(generator_version "9.0")
 	(paper "A3")
+	(rectangle
+		(start 267.97 43.18)
+		(end 326.39 256.54)
+		(stroke
+			(width 0)
+			(type default)
+			(color 255 0 252 1)
+		)
+		(fill
+			(type none)
+		)
+	)
+	(rectangle
+		(start 64.77 43.18)
+		(end 265.43 256.54)
+		(stroke
+			(width 0)
+			(type default)
+			(color 255 0 252 1)
+		)
+		(fill
+			(type none)
+		)
+	)
 	(text "Max 24V DC"
 		(exclude_from_sim no)
