File: IO_device.kicad_pcb (KiCad board)
At the start: 4 copper layers, 160 x 100 mm, 274 parts, among them J1 Screw_Terminal_01x02, J10 Screw_Terminal_01x02, J11 Screw_Terminal_01x02, J12 Screw_Terminal_01x02, J13 USB_C_Receptacle_PowerOnly_6P, J14 Conn_01x01, J15 Screw_Terminal_01x03, J17 Conn_01x01, J18 Conn_01x01, J19 Conn_01x01, J2 Screw_Terminal_01x02, J3 Screw_Terminal_01x02, J4 Screw_Terminal_01x02, J5 Screw_Terminal_01x02, J6 Screw_Terminal_01x02, J7 Screw_Terminal_01x02, J8 Screw_Terminal_01x02, J9 Screw_Terminal_01x02, K1 SDT-S-103DMR,000, K2 SDT-S-103DMR,000, K3 SDT-S-103DMR,000, K4 SDT-S-103DMR,000, Q1 BC847, Q11 BC847, Q12 BC847, Q13 AO3400A, Q2 BC847, Q3 BC847, Q4 BC847, Q5 2SCR587D3, Q6 2SCR587D3, Q7 AO3400A, Q8 AO3400A, Q9 AO3400A, U1 MCP4728, U10 74HC240D, U11 TL071, U12 TL071, U13 IL300-DEFG-X007T, U14 IL300-DEFG-X007T, U15 TL071, U16 TL071, U17 MCP3208T-BI/SL, U18 CNY173SR2VM, U19 CNY173SR2VM, U2 TL071, U20 CNY173SR2VM, U21 CNY173SR2VM, U22 MM74HC14M, U24 TBA1-0522E, U25 TBA1-0522E, U26 TBA1-0522E, U27 ADM2483xRW, U28 NUCLEO-L152RE, U3 TL071, U4 IL300-DEFG-X007T, U5 IL300-DEFG-X007T, U6 TL071, U7 TL071, U8 TL071, U9 TL071

Commit message: copper done
Routing:
- added copper zone on In1.Cu, net E5V
- added copper zone on B.Cu, net GNDD
- added copper zone on F.Cu, net GNDD
- added copper zone on In2.Cu, net GNDD
Changed lines of the file:
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@@
 		(net 232)
+	)
+	(zone
+		(net 1)
+		(net_name "GNDD")
+		(layer "F.Cu")
+		(hatch edge 0.5)
+		(connect_pads
+			(clearance 0.5)
+		)
+		(min_thickness 0.25)
+		(filled_areas_thickness no)
+		(fill yes
+			(thermal_gap 0.5)
+			(thermal_bridge_width 0.5)
+		)
+		(polygon
+			(pts
+				(xy 81.28 40.132) (xy 179.832 40.132) (xy 179.832 139.7) (xy 80.264 139.7)
+			)
+		)
+	)
+	(zone
+		(net 1)
+		(net_name "GNDD")
+		(layer "B.Cu")
+		(hatch edge 0.5)
+		(priority 2)
+		(connect_pads
+			(clearance 0.5)
+		)
+		(min_thickness 0.25)
+		(filled_areas_thickness no)
+		(fill yes
+			(thermal_gap 0.5)
+			(thermal_bridge_width 0.5)
+		)
+		(polygon
+			(pts
+				(xy 81.28 40.132) (xy 80.264 139.7) (xy 179.832 139.7) (xy 179.832 40.132)
+			)
+		)
+	)
+	(zone
+		(net 2)
+		(net_name "E5V")
+		(layer "In1.Cu")
+		(hatch edge 0.5)
+		(priority 3)
+		(connect_pads
+			(clearance 0.5)
+		)
+		(min_thickness 0.25)
+		(filled_areas_thickness no)
+		(fill yes
+			(thermal_gap 0.5)
+			(thermal_bridge_width 0.5)
+		)
+		(polygon
+			(pts
+				(xy 81.28 40.132) (xy 80.264 139.7) (xy 179.832 139.7) (xy 179.832 40.132)
+			)
+		)
+	)
+	(zone
+		(net 1)
+		(net_name "GNDD")
+		(layer "In2.Cu")
+		(hatch edge 0.5)
+		(priority 1)
+		(connect_pads
+			(clearance 0.5)
+		)
+		(min_thickness 0.25)
+		(filled_areas_thickness no)
+		(fill yes
+			(thermal_gap 0.5)
+			(thermal_bridge_width 0.5)
+		)
+		(polygon
+			(pts
+				(xy 81.28 40.132) (xy 80.264 139.7) (xy 179.832 139.7) (xy 179.832 40.132)
+			)
+		)
 	)
 	(embedded_fonts no)
